File: PCB/pathfinder.kicad_pcb (KiCad board)
At the start: 2 copper layers, 150 x 100 mm, 14 parts, among them SW1 SW_Push, SW2 SW_Push, SW3 SW_Push, SW4 SW_Push, SW5 SW_Push, SW6 SW_Push, SW7 SW_Push, SW8 SW_Push, SW9 SW_Push, U2 XIAO-RP2040-DIP

Commit message: Updates CAD
Parts:
- added H1: MountingHole, MountingHole:MountingHole_3.2mm_M3, F.Cu at (93.5, 68.5)
- added H2: MountingHole, MountingHole:MountingHole_3.2mm_M3, F.Cu at (231.5, 68.5)
- added H3: MountingHole, MountingHole:MountingHole_3.2mm_M3, F.Cu at (93.5, 137.0)
- added H4: MountingHole, MountingHole:MountingHole_3.2mm_M3, F.Cu at (231.5, 136.5)
