File: PCB/pathfinder.kicad_sch (KiCad schematic)
At the start: 14 parts, among them SW1 SW_Push, SW2 SW_Push, SW3 SW_Push, SW4 SW_Push, SW5 SW_Push, SW6 SW_Push, SW7 SW_Push, SW8 SW_Push, SW9 SW_Push, U2 XIAO-RP2040-DIP

Commit message: Updates CAD
Parts:
- added H1, H2, H3, H4: MountingHole, MountingHole:MountingHole_3.2mm_M3, symbol Mechanical:MountingHole

Commit message: pcb change
Connections:
- no-connect marks 0 -> 2
Changed lines of the file:
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@@
 	(generator_version "10.0")
 	(paper "A4")
+	(no_connect
+		(at 92.71 96.52)
+	)
+	(no_connect
+		(at 92.71 88.9)
+	)
 	(wire
 		(pts

Commit message: gerber and pcb
Parts:
- removed H1, H3: MountingHole, MountingHole:MountingHole_3.2mm_M3, symbol Mechanical:MountingHole
- added HSMALL1, HSMALL2: MountingHole, custom_footprints:mouse-bite-2mm-slot, symbol Mechanical:MountingHole
- added U3: XIAO-RP2040-DIP, footprints:XIAO-Generic-Hybrid-14P-2.54-21X17.8MM, symbol Seeed_Studio_XIAO_Series:XIAO-RP2040-DIP
- D1: value L08R5000Q1 -> POWER
- D2: value L08R5000Q1 -> Drift
- SW1: value SW_Push -> GAS
- SW2: value SW_Push -> BRAKE
- SW3: value SW_Push -> LEFT
- SW4: value SW_Push -> RIGHT
- SW5: value SW_Push -> CHECKPOINT
- SW6: value SW_Push -> RESTART
- SW7: value SW_Push -> AK40
- SW8: value SW_Push -> AK60
- SW9: value SW_Push -> AK80
- U2: footprint mito-keyboard mito-simplified main Seeed Studio XIAO Series Library:XIAO-RP2040-DIP -> footprints:XIAO-Generic-Hybrid-14P-2.54-21X17.8MM
- renumbered H2 to HBIG1, H4 to HBIG2
Connections:
- net AK40: now also U3.3 (GPIO28/ADC2/A2); no longer U2.7 (GPIO0/TX)
- net AK60: now also U2.5 (GPIO6/SDA); no longer U2.8 (GPIO1/RX)
- net AK80: now also U3.4 (GPIO29/ADC3/A3); no longer U2.9 (GPIO2/SCK)
- net CHECKPOINT: now also U3.1 (GPIO26/ADC0/A0); no longer U2.5 (GPIO6/SDA)
- net Drift Indicator: now also U3.5 (GPIO6/SDA); no longer U2.11 (GPIO3/MOSI)
- net GND: now also U3.13 (GND)
- net POWER: now also U2.6 (GPIO7/SCL); no longer U2.10 (GPIO4/MISO)
- net RESTART: now also U3.2 (GPIO27/ADC1/A1); no longer U2.6 (GPIO7/SCL)
Other:
- moved on the sheet: SW4, SW5, SW6, SW7, SW8, SW9

Commit message: prod, cad,
Parts:
- removed HSMALL1: MountingHole, custom_footprints:mouse-bite-2mm-slot, symbol Mechanical:MountingHole
Changed lines of the file:
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@@
-	)
-	(symbol
-		(lib_id "Mechanical:MountingHole")
-		(at 133.35 93.98 0)
-		(unit 1)
-		(body_style 1)
-		(exclude_from_sim no)
-		(in_bom no)
-		(on_board yes)
-		(in_pos_files yes)
-		(dnp no)
-		(fields_autoplaced yes)
-		(property "Reference" "HSMALL1"
-			(at 135.89 92.7099 0)
-			(show_name no)
-			(do_not_autoplace no)
-			(effects
-				(font
-					(size 1.27 1.27)
-				)
-				(justify left)
-			)
-		)
-		(property "Value" "MountingHole"
-			(at 135.89 95.2499 0)
-			(show_name no)
-			(do_not_autoplace no)
-			(effects
-				(font
-					(size 1.27 1.27)
-				)
-				(justify left)
-			)
-		)
-		(property "Footprint" "custom_footprints:mouse-bite-2mm-slot"
-			(at 133.35 93.98 0)
-			(hide yes)
-			(show_name no)
-			(do_not_autoplace no)
-			(effects
-				(font
-					(size 1.27 1.27)
-				)
-			)
-		)
-		(property "Datasheet" ""
-			(at 133.35 93.98 0)
-			(hide yes)
-			(show_name no)
-			(do_not_autoplace no)
-			(effects
-				(font
-					(size 1.27 1.27)
-				)
-			)
-		)
-		(property "Description" "Mounting Hole without connection"
-			(at 133.35 93.98 0)
-			(hide yes)
-			(show_name no)
-			(do_not_autoplace no)
-			(effects
-				(font
-					(size 1.27 1.27)
-				)
-			)
-		)
-		(instances
-			(project "pathfinder"
-				(path "/577f3b96-95aa-44e7-a29e-a89ce861cb4f"
-					(reference "HSMALL1")
-					(unit 1)
-				)
-			)
-		)
 	)
 	(symbol
